File: AV-board-robik/AV-board-robik.kicad_pcb (KiCad board)
At the start: 2 copper layers, 66 x 66 mm, 27 parts, among them J1 Mini-DIN-8, J2 Conn_01x09_Pin, Q1 BC547, Q2 BC547, Q3 BC547, Q4 BC547, U2 74LS241

Commit message: finished board
Parts:
- removed J1: Mini-DIN-8, w_conn_av:minidin-8
- removed J2: Conn_01x09_Pin, Connector_PinHeader_2.54mm:PinHeader_1x09_P2.54mm_Vertical
- added J3: Conn_01x09, Connector_PinHeader_2.54mm:PinHeader_1x09_P2.54mm_Horizontal, F.Cu at (120.4, 94.0)
- added J4: Conn_01x09, Connector_PinHeader_2.54mm:PinHeader_1x09_P2.54mm_Horizontal, F.Cu at (123.2, 94.0)
- moved R16 7.88 mm to (164.1, 58.7)
- moved R13 6.65 mm to (161.8, 111.8), turned to 0 degrees
- moved R14 6.65 mm to (161.8, 98.8), turned to 0 degrees
- moved R15 6.51 mm to (161.8, 85.9), turned to 0 degrees
- moved Q3 5.11 mm to (166.4, 89.7)
- moved R8 5.11 mm to (161.8, 76.2)
- moved C1 5.11 mm to (151.6, 64.0)
- moved Q1 5.11 mm to (166.4, 64.3)
- moved Q2 5.11 mm to (166.4, 77.2)
- moved Q4 5.11 mm to (166.4, 102.6)
- moved R10 5.11 mm to (161.8, 101.6)
- moved R11 5.11 mm to (161.8, 65.8)
- moved R12 5.11 mm to (161.8, 69.3)
- moved R6 5.11 mm to (161.8, 92.2)
- moved R9 5.11 mm to (161.8, 88.4)
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Connections:
- net Net-(D1-K) renamed /MD-2
- R11 pad 2: Net-(J1-Pad8) -> /MD-8
- R13 pad 2: Net-(J1-Pad7) -> /MD-7
- R14 pad 2: Net-(J1-Pad4) -> /MD-4
- R15 pad 2: Net-(J1-Pad6) -> /MD-6
- R16 pad 2: Net-(J1-Pad3) -> /MD-3
- RV1 pad 2: Net-(J1-Pad5) -> /MD-5
Routing:
- net /MD-4: track 0.00 -> 117.4 mm, vias 0 -> 4
- net /MD-6: track 0.00 -> 110.8 mm, vias 0 -> 4
- net /MD-8: track 0.00 -> 81.6 mm, vias 0 -> 4
- net /MD-7: track 0.00 -> 76.1 mm, vias 0 -> 2
- net /MD-3: track 0.00 -> 59.3 mm, vias 0 -> 2
- net GND: track 100.8 -> 160.0 mm, vias 4 -> 6
- net /+12V: track 0.00 -> 52.1 mm, vias 0 -> 2
- net /MD-2: track 4.06 -> 54.1 mm, vias 0 -> 2
- net /Y: track 0.00 -> 35.7 mm, vias 0 -> 2
- net /SYNC: track 0.00 -> 33.3 mm, vias 0 -> 2
- net /MD-5: track 0.00 -> 24.8 mm
- net /B: track 0.00 -> 22.5 mm, vias 0 -> 2
- net /AUDIO: track 0.00 -> 21.8 mm
- net /R: track 0.00 -> 20.6 mm, vias 0 -> 2
- net /G: track 0.00 -> 15.5 mm
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